Commit message: Update the gazebo UAV model to be the exact same with real machine.

File: jsk_uav_forest_simulation/urdf/quadrotor_cam_hokuyo.gazebo.xacro (robot description, xacro)
@@ -30,6 +30,6 @@
     <!-- Forward facing camera -->
     <xacro:include filename="$(find hector_sensors_description)/urdf/generic_camera.urdf.xacro" />
-    <xacro:generic_camera name="front_cam" parent="base_link" ros_topic="/camera/image" cam_info_topic="/camera/camera_info" update_rate="10" res_x="1280" res_y="1024" image_format="R8G8B8" hfov="100">
-      <origin xyz="0.2 0.0 0.0" rpy="0 0 0"/>
+    <xacro:generic_camera name="front_cam" parent="base_link" ros_topic="/camera/image" cam_info_topic="/camera/camera_info" update_rate="10" res_x="640" res_y="480" image_format="R8G8B8" hfov="54">
+      <origin xyz="0.0 0.0 0.15" rpy="0 0 0"/>
     </xacro:generic_camera>
     <xacro:include filename="$(find hector_quadrotor_gazebo)/urdf/quadrotor_plugins.gazebo.xacro" />
